File: PCB Design/microcontroller board/microcontroller board.kicad_sch (KiCad schematic)
At the start: 3 parts

Commit message: straight stick
Parts:
- added A4, A5, A6, A7, A8: Adafruit_Feather_Generic, Module:Adafruit_Feather, symbol MCU_Module:Adafruit_Feather_Generic
- gave numbers to parts that had none: 3
Connections:
- net at A1.17 (SDA), A2.17 (SDA), A3.17 (SDA): now also A1.4 (GND), A2.4 (GND), A3.4 (GND), A4.17 (SDA), A4.4 (GND), A5.17 (SDA), A5.4 (GND), A6.17 (SDA), A6.4 (GND), A7.17 (SDA), A7.4 (GND), A8.17 (SDA), A8.4 (GND)
- net at A1.18 (SCL), A2.18 (SCL), A3.18 (SCL): now also A4.18 (SCL), A5.18 (SCL), A6.18 (SCL), A7.18 (SCL), A8.18 (SCL)
- net at A1.2 (3V3), A2.2 (3V3), A3.2 (3V3): now also A4.2 (3V3), A5.2 (3V3), A6.2 (3V3), A7.2 (3V3), A8.2 (3V3)
Other:
- moved on the sheet: A1, A2, A3
