File: PCB Design/microcontroller mount/Adafruit NeoPixel 8 Stick.kicad_pcb (KiCad board)
At the start: 2 copper layers, 34.6 x 34 mm, 2 parts, among them CN2 1X4SMT, U1 DFR0282

Commit message: updates
Parts:
- added R-500_Ohm1: R, Resistor_THT:R_Axial_DIN0204_L3.6mm_D1.6mm_P7.62mm_Horizontal, F.Cu at (143.0, 125.0)
Connections:
- U1 pad A2: Net-(CN2-Pad3) -> Net-(R-500_Ohm1-Pad2)
Routing:
- net Net-(R-500_Ohm1-Pad2): track 0.00 -> 28.9 mm
- net Net-(CN2-Pad3): track 22.6 -> 44.6 mm
Other:
- board size 34.6 x 34 mm -> 34.6 x 37.8 mm
Changed lines of the file:
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@@
   (net 11 "unconnected-(U1-PadRX)")
   (net 12 "unconnected-(U1-PadTX)")
+  (net 13 "Net-(R-500_Ohm1-Pad2)")
+  (footprint "Resistor_THT:R_Axial_DIN0204_L3.6mm_D1.6mm_P7.62mm_Horizontal" (layer "F.Cu")
+    (at 143.002 124.968 180)
+    (descr "Resistor, Axial_DIN0204 series, Axial, Horizontal, pin pitch=7.62mm, 0.167W, length*diameter=3.6*1.6mm^2, http://cdn-reichelt.de/documents/datenblatt/B400/1_4W%23YAG.pdf")
+    (tags "Resistor Axial_DIN0204 series Axial Horizontal pin pitch 7.62mm 0.167W length 3.6mm diameter 1.6mm")
+    (property "Sheetfile" "Adafruit NeoPixel 8 Stick.kicad_sch")
+    (property "Sheetname" "")
+    (attr through_hole)
+    (fp_text reference "R-500_Ohm1" (at 3.81 -1.92) (layer "F.SilkS")
+      (effects (font (size 1 1) (thickness 0.15)))
+    )
+    (fp_text value "R" (at 3.81 1.92) (layer "F.Fab")
+      (effects (font (size 1 1) (thickness 0.15)))
+    )
+    (fp_text user "${REFERENCE}" (at 3.81 0) (layer "F.Fab")
+      (effects (font (size 0.72 0.72) (thickness 0.108)))
+    )
+    (fp_line (start 0.94 0) (end 1.89 0) (layer "F.SilkS") (width 0.12))
+    (fp_line (start 1.89 0.92) (end 5.73 0.92) (layer "F.SilkS") (width 0.12))
+    (fp_line (start 6.68 0) (end 5.73 0) (layer "F.SilkS") (width 0.12))
+    (fp_line (start 1.89 -0.92) (end 1.89 0.92) (layer "F.SilkS") (width 0.12))
+    (fp_line (start 5.73 -0.92) (end 1.89 -0.92) (layer "F.SilkS") (width 0.12))
+    (fp_line (start 5.73 0.92) (end 5.73 -0.92) (layer "F.SilkS") (width 0.12))
+    (fp_line (start 8.57 1.05) (end 8.57 -1.05) (layer "F.CrtYd") (width 0.05))
+    (fp_line (start -0.95 -1.05) (end -0.95 1.05) (layer "F.CrtYd") (width 0.05))
+    (fp_line (start -0.95 1.05) (end 8.57 1.05) (layer "F.CrtYd") (width 0.05))
+    (fp_line (start 8.57 -1.05) (end -0.95 -1.05) (layer "F.CrtYd") (width 0.05))
+    (fp_line (start 5.61 -0.8) (end 2.01 -0.8) (layer "F.Fab") (width 0.1))
+    (fp_line (start 7.62 0) (end 5.61 0) (layer "F.Fab") (width 0.1))
+    (fp_line (start 5.61 0.8) (end 5.61 -0.8) (layer "F.Fab") (width 0.1))
+    (fp_line (start 2.01 -0.8) (end 2.01 0.8) (layer "F.Fab") (width 0.1))
+    (fp_line (start 2.01 0.8) (end 5.61 0.8) (layer "F.Fab") (width 0.1))
+    (fp_line (start 0 0) (end 2.01 0) (layer "F.Fab") (width 0.1))
+    (pad "1" thru_hole circle (at 0 0 180) (size 1.4 1.4) (drill 0.7) (layers *.Cu *.Mask)
+      (net 3 "Net-(CN2-Pad3)") (pintype "passive"))
+    (pad "2" thru_hole oval (at 7.62 0 180) (size 1.4 1.4) (drill 0.7) (layers *.Cu *.Mask)
+      (net 13 "Net-(R-500_Ohm1-Pad2)") (pintype "passive"))
+    (model "${KICAD6_3DMODEL_DIR}/Resistor_THT.3dshapes/R_Axial_DIN0204_L3.6mm_D1.6mm_P7.62mm_Horizontal.wrl"
+      (offset (xyz 0 0 0))
+      (scale (xyz 1 1 1))
+      (rotate (xyz 0 0 0))
+    )
+  )
   (footprint "DFR0282:DFR0282" (layer "F.Cu")
     (at 139.954 108.458)
@@
       (effects (font (size 1 1) (thickness 0.15)))
     )
+    (fp_text user "_" (at -13.2 -8.3) (layer "F.Fab")
+      (effects (font (size 1 1) (thickness 0.15)))
+    )
     (fp_text user "+" (at 12 -7.3) (layer "F.Fab")
       (effects (font (size 1 1) (thickness 0.15)))
     )
-    (fp_text user "_" (at -13.2 -8.3) (layer "F.Fab")
-      (effects (font (size 1 1) (thickness 0.15)))
-    )
     (fp_line (start 10 11.25) (end 10 8.85) (layer "F.SilkS") (width 0.127))
+    (fp_line (start -10 -11.25) (end 10 -11.25) (layer "F.SilkS") (width 0.127))
+    (fp_line (start -10 11.25) (end -5.55 11.25) (layer "F.SilkS") (width 0.127))
     (fp_line (start 10 -11.25) (end 10 -10.3) (layer "F.SilkS") (width 0.127))
     (fp_line (start -10 -10.3) (end -10 -11.25) (layer "F.SilkS") (width 0.127))
-    (fp_line (start -10 -11.25) (end 10 -11.25) (layer "F.SilkS") (width 0.127))
     (fp_line (start 5.55 11.25) (end 10 11.25) (layer "F.SilkS") (width 0.127))
     (fp_line (start -10 8.85) (end -10 11.25) (layer "F.SilkS") (width 0.127))
-    (fp_line (start -10 11.25) (end -5.55 11.25) (layer "F.SilkS") (width 0.127))
+    (fp_line (start 11.65 -11.5) (end 11.65 12.9) (layer "F.CrtYd") (width 0.05))
     (fp_line (start -11.65 -11.5) (end 11.65 -11.5) (layer "F.CrtYd") (width 0.05))
-    (fp_line (start 11.65 -11.5) (end 11.65 12.9) (layer "F.CrtYd") (width 0.05))
     (fp_line (start -11.65 12.9) (end 11.65 12.9) (layer "F.CrtYd") (width 0.05))
     (fp_line (start -11.65 -11.5) (end -11.65 12.9) (layer "F.CrtYd") (width 0.05))
     (fp_line (start 10 11.25) (end -10 11.25) (layer "F.Fab") (width 0.127))
+    (fp_line (start 10 -11.25) (end 10 11.25) (layer "F.Fab") (width 0.127))
+    (fp_line (start -10 -11.25) (end 10 -11.25) (layer "F.Fab") (width 0.127))
     (fp_line (start -10 11.25) (end -10 -11.25) (layer "F.Fab") (width 0.127))
-    (fp_line (start -10 -11.25) (end 10 -11.25) (layer "F.Fab") (width 0.127))
-    (fp_line (start 10 -11.25) (end 10 11.25) (layer "F.Fab") (width 0.127))
     (pad "A0" smd rect (at 8.9 6.5) (size 5 3.5) (layers "F.Cu" "F.Paste" "F.Mask")
       (net 6 "unconnected-(U1-PadA0)") (pinfunction "A0") (pintype "bidirectional"))
@@
       (net 7 "unconnected-(U1-PadA1)") (pinfunction "A1") (pintype "bidirectional"))
     (pad "A2" smd rect (at 8.9 -3.1) (size 5 3.5) (layers "F.Cu" "F.Paste" "F.Mask")
-      (net 3 "Net-(CN2-Pad3)") (pinfunction "A2") (pintype "bidirectional"))
+      (net 13 "Net-(R-500_Ohm1-Pad2)") (pinfunction "A2") (pintype "bidirectional"))
     (pad "D9" smd rect (at -8.9 6.5) (size 5 3.5) (layers "F.Cu" "F.Paste" "F.Mask")
       (net 8 "unconnected-(U1-PadD9)") (pinfunction "D9") (pintype "bidirectional"))
@@
   )
   (gr_line (start 130.048 89.915998) (end 149.352 89.915999) (layer "Edge.Cuts") (width 0.05))
-  (gr_line (start 122.428 97.536) (end 122.428 123.952) (layer "Edge.Cuts") (width 0.05))
+  (gr_line (start 122.428 97.536) (end 122.428 127.762) (layer "Edge.Cuts") (width 0.05))
   (gr_line (start 149.352 89.915999) (end 156.972 97.45) (layer "Edge.Cuts") (width 0.05))
-  (gr_line (start 122.428 123.952) (end 157.054 123.952) (layer "Edge.Cuts") (width 0.05))
-  (gr_line (start 156.972 97.45) (end 157.054 123.952) (layer "Edge.Cuts") (width 0.05))
+  (gr_line (start 122.428 127.762) (end 157.054 127.762) (layer "Edge.Cuts") (width 0.05))
+  (gr_line (start 156.972 97.45) (end 157.054 127.762) (layer "Edge.Cuts") (width 0.05))
   (gr_line (start 122.428 97.536) (end 130.048 89.915998) (layer "Edge.Cuts") (width 0.05))
   (segment (start 148.854 98.562) (end 144.145 93.853) (width 0.25) (layer "F.Cu") (net 1))
@@
   (via (at 131.064 100.584) (size 0.8) (drill 0.4) (layers "F.Cu" "B.Cu") (net 2))
   (via (at 143.256 118.618) (size 0.8) (drill 0.4) (layers "F.Cu" "B.Cu") (net 2))
-  (segment (start 146.045322 92.202) (end 140.97 92.202) (width 0.25) (layer "F.Cu") (net 3))
-  (segment (start 152.1354 102.8266) (end 152.1354 98.292078) (width 0.25) (layer "F.Cu") (net 3))
-  (segment (start 149.604 105.358) (end 152.1354 102.8266) (width 0.25) (layer "F.Cu") (net 3))
-  (segment (start 152.1354 98.292078) (end 146.045322 92.202) (width 0.25) (layer "F.Cu") (net 3))
-  (segment (start 148.854 105.358) (end 149.604 105.358) (width 0.25) (layer "F.Cu") (net 3))
+  (segment (start 152.146 98.302678) (end 152.146 116.586) (width 0.25) (layer "F.Cu") (net 3))
+  (segment (start 143.764 124.968) (end 143.002 124.968) (width 0.25) (layer "F.Cu") (net 3))
+  (segment (start 146.045322 92.202) (end 152.146 98.302678) (width 0.25) (layer "F.Cu") (net 3))
+  (segment (start 152.146 116.586) (end 143.764 124.968) (width 0.25) (layer "F.Cu") (net 3))
+  (segment (start 140.97 92.202) (end 146.045322 92.202) (width 0.25) (layer "F.Cu") (net 3))
   (via (at 140.97 92.202) (size 0.8) (drill 0.4) (layers "F.Cu" "B.Cu") (net 3))
   (segment (start 128.2258 117.1538) (end 128.2258 98.5962) (width 0.25) (layer "F.Cu") (net 4))
@@
   (segment (start 151.6822 102.6362) (end 151.6822 98.4798) (width 0.25) (layer "F.Cu") (net 5))
   (via (at 131.826 93.726) (size 0.8) (drill 0.4) (layers "F.Cu" "B.Cu") (net 5))
+  (segment (start 148.854 105.358) (end 146.0258 108.1862) (width 0.25) (layer "F.Cu") (net 13))
+  (segment (start 143.51 123.19) (end 137.16 123.19) (width 0.25) (layer "F.Cu") (net 13))
+  (segment (start 137.16 123.19) (end 135.382 124.968) (width 0.25) (layer "F.Cu") (net 13))
+  (segment (start 146.0258 108.1862) (end 146.0258 120.6742) (width 0.25) (layer "F.Cu") (net 13))
+  (segment (start 146.0258 120.6742) (end 143.51 123.19) (width 0.25) (layer "F.Cu") (net 13))
   (zone (net 2) (net_name "GND") (layers F&B.Cu) (hatch edge 0.508)
     (connect_pads (clearance 0.000001))
@@
     (polygon
       (pts
-        (xy 160.02 126.492)
-        (xy 119.634 126.492)
+        (xy 160.02 150.368)
+        (xy 119.634 150.368)
         (xy 119.634 85.852)
         (xy 160.02 85.852)

Commit message: updates
Connections:
- U1 pad A2: Net-(R-500_Ohm1-Pad2) -> unconnected-(U1-PadA2)
- U1 pad D10: unconnected-(U1-PadD10) -> Net-(R-500_Ohm1-Pad2)
Routing:
- net Net-(R-500_Ohm1-Pad2): track 28.9 -> 16.5 mm, vias 0 -> 1
Changed lines of the file:
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@@
   (net 7 "unconnected-(U1-PadA1)")
   (net 8 "unconnected-(U1-PadD9)")
-  (net 9 "unconnected-(U1-PadD10)")
-  (net 10 "unconnected-(U1-PadD11)")
-  (net 11 "unconnected-(U1-PadRX)")
-  (net 12 "unconnected-(U1-PadTX)")
-  (net 13 "Net-(R-500_Ohm1-Pad2)")
+  (net 9 "unconnected-(U1-PadD11)")
+  (net 10 "unconnected-(U1-PadRX)")
+  (net 11 "unconnected-(U1-PadTX)")
+  (net 12 "Net-(R-500_Ohm1-Pad2)")
+  (net 13 "unconnected-(U1-PadA2)")
   (footprint "Resistor_THT:R_Axial_DIN0204_L3.6mm_D1.6mm_P7.62mm_Horizontal" (layer "F.Cu")
     (at 143.002 124.968 180)
@@
       (net 3 "Net-(CN2-Pad3)") (pintype "passive"))
     (pad "2" thru_hole oval (at 7.62 0 180) (size 1.4 1.4) (drill 0.7) (layers *.Cu *.Mask)
-      (net 13 "Net-(R-500_Ohm1-Pad2)") (pintype "passive"))
+      (net 12 "Net-(R-500_Ohm1-Pad2)") (pintype "passive"))
     (model "${KICAD6_3DMODEL_DIR}/Resistor_THT.3dshapes/R_Axial_DIN0204_L3.6mm_D1.6mm_P7.62mm_Horizontal.wrl"
       (offset (xyz 0 0 0))
@@
       (effects (font (size 1 1) (thickness 0.15)))
     )
+    (fp_text user "+" (at 12 -7.3) (layer "F.SilkS")
+      (effects (font (size 1 1) (thickness 0.15)))
+    )
     (fp_text user "_" (at -13.2 -8.3) (layer "F.SilkS")
       (effects (font (size 1 1) (thickness 0.15)))
     )
-    (fp_text user "+" (at 12 -7.3) (layer "F.SilkS")
+    (fp_text user "+" (at 12 -7.3) (layer "F.Fab")
       (effects (font (size 1 1) (thickness 0.15)))
     )
@@
       (effects (font (size 1 1) (thickness 0.15)))
     )
-    (fp_text user "+" (at 12 -7.3) (layer "F.Fab")
-      (effects (font (size 1 1) (thickness 0.15)))
-    )
+    (fp_line (start -10 8.85) (end -10 11.25) (layer "F.SilkS") (width 0.127))
+    (fp_line (start 5.55 11.25) (end 10 11.25) (layer "F.SilkS") (width 0.127))
+    (fp_line (start 10 -11.25) (end 10 -10.3) (layer "F.SilkS") (width 0.127))
     (fp_line (start 10 11.25) (end 10 8.85) (layer "F.SilkS") (width 0.127))
     (fp_line (start -10 -11.25) (end 10 -11.25) (layer "F.SilkS") (width 0.127))
     (fp_line (start -10 11.25) (end -5.55 11.25) (layer "F.SilkS") (width 0.127))
-    (fp_line (start 10 -11.25) (end 10 -10.3) (layer "F.SilkS") (width 0.127))
     (fp_line (start -10 -10.3) (end -10 -11.25) (layer "F.SilkS") (width 0.127))
-    (fp_line (start 5.55 11.25) (end 10 11.25) (layer "F.SilkS") (width 0.127))
-    (fp_line (start -10 8.85) (end -10 11.25) (layer "F.SilkS") (width 0.127))
+    (fp_line (start -11.65 -11.5) (end -11.65 12.9) (layer "F.CrtYd") (width 0.05))
+    (fp_line (start -11.65 -11.5) (end 11.65 -11.5) (layer "F.CrtYd") (width 0.05))
     (fp_line (start 11.65 -11.5) (end 11.65 12.9) (layer "F.CrtYd") (width 0.05))
-    (fp_line (start -11.65 -11.5) (end 11.65 -11.5) (layer "F.CrtYd") (width 0.05))
     (fp_line (start -11.65 12.9) (end 11.65 12.9) (layer "F.CrtYd") (width 0.05))
-    (fp_line (start -11.65 -11.5) (end -11.65 12.9) (layer "F.CrtYd") (width 0.05))
+    (fp_line (start 10 -11.25) (end 10 11.25) (layer "F.Fab") (width 0.127))
     (fp_line (start 10 11.25) (end -10 11.25) (layer "F.Fab") (width 0.127))
-    (fp_line (start 10 -11.25) (end 10 11.25) (layer "F.Fab") (width 0.127))
     (fp_line (start -10 -11.25) (end 10 -11.25) (layer "F.Fab") (width 0.127))
     (fp_line (start -10 11.25) (end -10 -11.25) (layer "F.Fab") (width 0.127))
@@
       (net 7 "unconnected-(U1-PadA1)") (pinfunction "A1") (pintype "bidirectional"))
     (pad "A2" smd rect (at 8.9 -3.1) (size 5 3.5) (layers "F.Cu" "F.Paste" "F.Mask")
-      (net 13 "Net-(R-500_Ohm1-Pad2)") (pinfunction "A2") (pintype "bidirectional"))
+      (net 13 "unconnected-(U1-PadA2)") (pinfunction "A2") (pintype "bidirectional"))
     (pad "D9" smd rect (at -8.9 6.5) (size 5 3.5) (layers "F.Cu" "F.Paste" "F.Mask")
       (net 8 "unconnected-(U1-PadD9)") (pinfunction "D9") (pintype "bidirectional"))
     (pad "D10" smd rect (at -8.9 1.7) (size 5 3.5) (layers "F.Cu" "F.Paste" "F.Mask")
-      (net 9 "unconnected-(U1-PadD10)") (pinfunction "D10") (pintype "bidirectional"))
+      (net 12 "Net-(R-500_Ohm1-Pad2)") (pinfunction "D10") (pintype "bidirectional"))
     (pad "D11" smd rect (at -8.9 -3.1) (size 5 3.5) (layers "F.Cu" "F.Paste" "F.Mask")
-      (net 10 "unconnected-(U1-PadD11)") (pinfunction "D11") (pintype "bidirectional"))
+      (net 9 "unconnected-(U1-PadD11)") (pinfunction "D11") (pintype "bidirectional"))
     (pad "GND1" smd rect (at -8.9 -7.9) (size 5 3.5) (layers "F.Cu" "F.Paste" "F.Mask")
       (net 2 "GND") (pinfunction "GND") (pintype "power_in"))
@@
       (net 2 "GND") (pinfunction "GND") (pintype "power_in"))
     (pad "RX" smd rect (at -3.5 4.75) (size 3 3) (layers "F.Cu" "F.Paste" "F.Mask")
-      (net 11 "unconnected-(U1-PadRX)") (pinfunction "RX") (pintype "input"))
+      (net 10 "unconnected-(U1-PadRX)") (pinfunction "RX") (pintype "input"))
     (pad "SCL" smd rect (at 3.5 -0.75) (size 3 3) (layers "F.Cu" "F.Paste" "F.Mask")
       (net 5 "Net-(CN2-Pad6)") (pinfunction "SCL") (pintype "input"))
@@
       (net 4 "Net-(CN2-Pad5)") (pinfunction "SDA") (pintype "bidirectional"))
     (pad "TX" smd rect (at -3.5 -0.75) (size 3 3) (layers "F.Cu" "F.Paste" "F.Mask")
-      (net 12 "unconnected-(U1-PadTX)") (pinfunction "TX") (pintype "output"))
+      (net 11 "unconnected-(U1-PadTX)") (pinfunction "TX") (pintype "output"))
     (pad "VCC1" smd rect (at 8.9 -7.9) (size 5 3.5) (layers "F.Cu" "F.Paste" "F.Mask")
       (net 1 "+5V") (pinfunction "VCC") (pintype "power_in"))
@@
   (segment (start 151.6822 102.6362) (end 151.6822 98.4798) (width 0.25) (layer "F.Cu") (net 5))
   (via (at 131.826 93.726) (size 0.8) (drill 0.4) (layers "F.Cu" "B.Cu") (net 5))
-  (segment (start 148.854 105.358) (end 146.0258 108.1862) (width 0.25) (layer "F.Cu") (net 13))
-  (segment (start 143.51 123.19) (end 137.16 123.19) (width 0.25) (layer "F.Cu") (net 13))
-  (segment (start 137.16 123.19) (end 135.382 124.968) (width 0.25) (layer "F.Cu") (net 13))
-  (segment (start 146.0258 108.1862) (end 146.0258 120.6742) (width 0.25) (layer "F.Cu") (net 13))
-  (segment (start 146.0258 120.6742) (end 143.51 123.19) (width 0.25) (layer "F.Cu") (net 13))
+  (via (at 131.064 110.236) (size 0.8) (drill 0.4) (layers "F.Cu" "B.Cu") (net 12))
+  (segment (start 135.382 124.968) (end 135.382 114.554) (width 0.25) (layer "B.Cu") (net 12))
+  (segment (start 135.382 114.554) (end 131.064 110.236) (width 0.25) (layer "B.Cu") (net 12))
   (zone (net 2) (net_name "GND") (layers F&B.Cu) (hatch edge 0.508)
     (connect_pads (clearance 0.000001))
