File: PCB Design/microcontroller mount/Adafruit NeoPixel 8 Stick.kicad_pcb (KiCad board)
At the start: 2 copper layers, 34.6 x 37.8 mm, 3 parts, among them CN2 1X4SMT, U1 DFR0282

Commit message: changes
Parts:
- added R1: R, Resistor_THT:R_Axial_DIN0207_L6.3mm_D2.5mm_P7.62mm_Horizontal, F.Cu at (146.8, 125.0)
- added U2: MIC5219-2.8YM5, Package_TO_SOT_SMD:SOT-23-5, F.Cu at (130.6, 125.0)
- added U3: VL6180, Adafruit VL6180 Time of Flight Sensor:VL6180, F.Cu at (125.5, 124.2)
- R-500_Ohm1: footprint Resistor_THT:R_Axial_DIN0204_L3.6mm_D1.6mm_P7.62mm_Horizontal -> Resistor_THT:R_Axial_DIN0207_L6.3mm_D2.5mm_P7.62mm_Horizontal
Routing:
- net Net-(CN2-Pad5): track 49.4 -> 86.8 mm, vias 1 -> 2
- net Net-(CN2-Pad6): track 38.3 -> 73.3 mm
- net Net-(R1-Pad2): track 0.00 -> 35.0 mm
- net Net-(R1-Pad1): track 0.00 -> 34.2 mm, vias 0 -> 1
- net GND: track 0.00 -> 19.3 mm
- net +5V: track 33.3 -> 48.3 mm, vias 1 -> 4
Other:
- board size 34.6 x 37.8 mm -> 34.6 x 38.4 mm

Commit message: argon mount
Parts:
- removed R1: R, Resistor_THT:R_Axial_DIN0207_L6.3mm_D2.5mm_P7.62mm_Horizontal
- removed U2: MIC5219-2.8YM5, Package_TO_SOT_SMD:SOT-23-5
- removed U3: VL6180, Adafruit VL6180 Time of Flight Sensor:VL6180
Routing:
- net Net-(CN2-Pad5): track 86.8 -> 49.4 mm, vias 2 -> 1
- net Net-(CN2-Pad6): track 73.3 -> 38.3 mm
- net Net-(R1-Pad2): track 35.0 -> 0.00 mm
- net Net-(R1-Pad1): track 34.2 -> 0.00 mm, vias 1 -> 0
- net GND: track 19.3 -> 0.00 mm
- net +5V: track 48.3 -> 31.2 mm, vias 4 -> 1
