File: PCB Design/power/Adafruit NeoPixel 8 Stick.kicad_sch (KiCad schematic)
At the start: 2 parts, among them CN2 1X4SMT

Commit message: finished power supply
Parts:
- added J1: PJ-102AH, PJ-102AH:PJ-102AH, symbol PJ-102AH:PJ-102AH
Connections:
- net +5V: now also J1.1
- net GND: now also J1.2
Changed lines of the file:
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@@
     (pin "1")
+  )
+  (symbol (lib_id "PJ-102AH:PJ-102AH") (at 64.77 123.19 180) (unit 1)
+    (in_bom yes) (on_board yes) (fields_autoplaced)
+    (property "Reference" "J1" (id 0) (at 73.66 122.8724 0)
+      (effects (font (size 1.27 1.27)) (justify right))
+    )
+    (property "Value" "PJ-102AH" (id 1) (at 73.66 125.4124 0)
+      (effects (font (size 1.27 1.27)) (justify right))
+    )
+    (property "Footprint" "PJ-102AH:PJ-102AH" (id 2) (at 69.85 129.54 0)
+      (effects (font (size 1.27 1.27)) (justify left bottom) hide)
+    )
+    (property "Datasheet" "" (id 3) (at 64.77 123.19 0)
+      (effects (font (size 1.27 1.27)) (justify left bottom) hide)
+    )
+    (property "STANDARD" "" (id 4) (at 71.12 132.08 0)
+      (effects (font (size 1.27 1.27)) (justify left bottom) hide)
+    )
+    (property "PART_REV" "" (id 5) (at 71.12 133.35 0)
+      (effects (font (size 1.27 1.27)) (justify left bottom) hide)
+    )
+    (property "MANUFACTURER" "" (id 6) (at 66.04 133.35 0)
+      (effects (font (size 1.27 1.27)) (justify left bottom) hide)
+    )
+    (pin "1")
+    (pin "2")
+    (pin "3")
   )
   (symbol (lib_id "Adafruit NeoPixel 8 Stick-eagle-import:GND") (at 45.72 138.43 0) (unit 1)
@@
     (pin "6")
   )
+  (symbol (lib_id "Adafruit NeoPixel 8 Stick-eagle-import:+5V") (at 59.69 128.27 180) (unit 1)
+    (in_bom yes) (on_board yes)
+    (property "Reference" "#P+0101" (id 0) (at 59.69 128.27 0)
+      (effects (font (size 1.27 1.27)) hide)
+    )
+    (property "Value" "+5V" (id 1) (at 62.23 123.19 90)
+      (effects (font (size 1.778 1.5113)) (justify left bottom))
+    )
+    (property "Footprint" "Adafruit NeoPixel 8 Stick:" (id 2) (at 59.69 128.27 0)
+      (effects (font (size 1.27 1.27)) hide)
+    )
+    (property "Datasheet" "" (id 3) (at 59.69 128.27 0)
+      (effects (font (size 1.27 1.27)) hide)
+    )
+    (pin "1")
+  )
+  (symbol (lib_id "Adafruit NeoPixel 8 Stick-eagle-import:GND") (at 59.69 118.11 180) (unit 1)
+    (in_bom yes) (on_board yes)
+    (property "Reference" "#SUPPLY0102" (id 0) (at 59.69 118.11 0)
+      (effects (font (size 1.27 1.27)) hide)
+    )
+    (property "Value" "GND" (id 1) (at 62.23 114.3 0)
+      (effects (font (size 1.778 1.5113)) (justify left bottom))
+    )
+    (property "Footprint" "Adafruit NeoPixel 8 Stick:" (id 2) (at 59.69 118.11 0)
+      (effects (font (size 1.27 1.27)) hide)
+    )
+    (property "Datasheet" "" (id 3) (at 59.69 118.11 0)
+      (effects (font (size 1.27 1.27)) hide)
+    )
+    (pin "1")
+  )
   (symbol (lib_id "Device:C_Polarized") (at 49.53 130.81 270) (unit 1)
     (in_bom yes) (on_board yes) (fields_autoplaced)
@@
   )
   (symbol_instances
+    (path "/721af9eb-87b4-40a0-a972-75811b7b9f2a"
+      (reference "#P+0101") (unit 1) (value "+5V") (footprint "Adafruit NeoPixel 8 Stick:")
+    )
     (path "/37ba77a5-6ca2-4fbe-a6d2-b4abdc4b9fc5"
       (reference "#P+0102") (unit 1) (value "+5V") (footprint "Adafruit NeoPixel 8 Stick:")
@@
       (reference "#SUPPLY0101") (unit 1) (value "GND") (footprint "Adafruit NeoPixel 8 Stick:")
     )
+    (path "/fc3bba3e-6c7d-4d86-9b14-bacaf910f85e"
+      (reference "#SUPPLY0102") (unit 1) (value "GND") (footprint "Adafruit NeoPixel 8 Stick:")
+    )
     (path "/fd13b4de-5fec-4ab3-89d0-81927074ae16"
       (reference "C1") (unit 1) (value "C_Polarized") (footprint "Capacitor_THT:CP_Radial_D12.5mm_P6.00mm")
@@
       (reference "CN2") (unit 1) (value "1X4SMT") (footprint "Adafruit NeoPixel 8 Stick:1X4-SMT")
     )
+    (path "/3cb3a231-372a-4344-831b-75ae89c16824"
+      (reference "J1") (unit 1) (value "PJ-102AH") (footprint "PJ-102AH:PJ-102AH")
+    )
   )
