File: PCB Design/T intersection straight/Adafruit NeoPixel 8 Stick.kicad_pcb (KiCad board)
At the start: 2 copper layers, 36.6 x 28.6 mm, 8 parts, among them CN1 1X4SMT, CN2 1X4SMT, CN3 1X4SMT

Commit message: changes
Connections:
- CN3 pad 1: unconnected-(CN3-Pad1) -> Net-(CN1-Pad1)
- CN3 pad 2: unconnected-(CN3-Pad2) -> Net-(CN1-Pad2)
Routing:
- net Net-(CN1-Pad2): track 29.7 -> 53.3 mm
- net Net-(CN1-Pad1): track 29.7 -> 40.0 mm
Changed lines of the file:
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@@
   (net 5 "+5V")
   (net 6 "Net-(CN2-Pad3)")
-  (net 7 "unconnected-(CN3-Pad1)")
-  (net 8 "unconnected-(CN3-Pad2)")
-  (net 9 "Net-(CN3-Pad3)")
-  (net 10 "Net-(CN3-Pad4)")
-  (net 11 "Net-(D1-Pad2)")
-  (net 12 "Net-(D3-Pad2)")
-  (net 13 "Net-(D7-Pad4)")
+  (net 7 "Net-(D6-Pad2)")
+  (net 8 "Net-(CN3-Pad3)")
+  (net 9 "Net-(CN3-Pad4)")
+  (net 10 "Net-(D1-Pad2)")
+  (net 11 "Net-(D3-Pad2)")
   (footprint "LED_SMD:LED_WS2812B_PLCC4_5.0x5.0mm_P3.2mm" (layer "F.Cu")
     (at 146.558 102.616 135)
@@
       (net 1 "GND") (pinfunction "VDD") (pintype "power_in"))
     (pad "2" smd rect (at -2.45 1.6 135) (size 1.5 1) (layers "F.Cu" "F.Paste" "F.Mask")
-      (net 13 "Net-(D7-Pad4)") (pinfunction "DOUT") (pintype "output"))
+      (net 7 "Net-(D6-Pad2)") (pinfunction "DOUT") (pintype "output"))
     (pad "3" smd rect (at 2.45 1.6 135) (size 1.5 1) (layers "F.Cu" "F.Paste" "F.Mask")
       (net 5 "+5V") (pinfunction "VSS") (pintype "power_in"))
     (pad "4" smd rect (at 2.45 -1.6 135) (size 1.5 1) (layers "F.Cu" "F.Paste" "F.Mask")
-      (net 12 "Net-(D3-Pad2)") (pinfunction "DIN") (pintype "input"))
+      (net 11 "Net-(D3-Pad2)") (pinfunction "DIN") (pintype "input"))
     (model "${KICAD6_3DMODEL_DIR}/LED_SMD.3dshapes/LED_WS2812B_PLCC4_5.0x5.0mm_P3.2mm.wrl"
       (offset (xyz 0 0 0))
@@
       (net 5 "+5V") (pinfunction "VDD") (pintype "power_in"))
     (pad "2" smd rect (at -2.45 1.6 180) (size 1.5 1) (layers "F.Cu" "F.Paste" "F.Mask")
-      (net 11 "Net-(D1-Pad2)") (pinfunction "DOUT") (pintype "output"))
+      (net 10 "Net-(D1-Pad2)") (pinfunction "DOUT") (pintype "output"))
     (pad "3" smd rect (at 2.45 1.6 180) (size 1.5 1) (layers "F.Cu" "F.Paste" "F.Mask")
       (net 1 "GND") (pinfunction "VSS") (pintype "power_in"))
@@
       (net 5 "+5V") (pinfunction "VDD") (pintype "power_in"))
     (pad "2" smd rect (at -2.45 1.6 90) (size 1.5 1) (layers "F.Cu" "F.Paste" "F.Mask")
-      (net 9 "Net-(CN3-Pad3)") (pinfunction "DOUT") (pintype "output"))
+      (net 8 "Net-(CN3-Pad3)") (pinfunction "DOUT") (pintype "output"))
     (pad "3" smd rect (at 2.45 1.6 90) (size 1.5 1) (layers "F.Cu" "F.Paste" "F.Mask")
       (net 1 "GND") (pinfunction "VSS") (pintype "power_in"))
     (pad "4" smd rect (at 2.45 -1.6 90) (size 1.5 1) (layers "F.Cu" "F.Paste" "F.Mask")
-      (net 10 "Net-(CN3-Pad4)") (pinfunction "DIN") (pintype "input"))
+      (net 9 "Net-(CN3-Pad4)") (pinfunction "DIN") (pintype "input"))
     (model "${KICAD6_3DMODEL_DIR}/LED_SMD.3dshapes/LED_WS2812B_PLCC4_5.0x5.0mm_P3.2mm.wrl"
       (offset (xyz 0 0 0))
@@
       (net 5 "+5V") (pinfunction "VSS") (pintype "power_in"))
     (pad "4" smd rect (at 2.45 -1.6 180) (size 1.5 1) (layers "F.Cu" "F.Paste" "F.Mask")
-      (net 13 "Net-(D7-Pad4)") (pinfunction "DIN") (pintype "input"))
+      (net 7 "Net-(D6-Pad2)") (pinfunction "DIN") (pintype "input"))
     (model "${KICAD6_3DMODEL_DIR}/LED_SMD.3dshapes/LED_WS2812B_PLCC4_5.0x5.0mm_P3.2mm.wrl"
       (offset (xyz 0 0 0))
@@
       (net 1 "GND") (pinfunction "VDD") (pintype "power_in"))
     (pad "2" smd rect (at -2.45 1.6 225) (size 1.5 1) (layers "F.Cu" "F.Paste" "F.Mask")
-      (net 12 "Net-(D3-Pad2)") (pinfunction "DOUT") (pintype "output"))
+      (net 11 "Net-(D3-Pad2)") (pinfunction "DOUT") (pintype "output"))
     (pad "3" smd rect (at 2.45 1.6 225) (size 1.5 1) (layers "F.Cu" "F.Paste" "F.Mask")
       (net 5 "+5V") (pinfunction "VSS") (pintype "power_in"))
     (pad "4" smd rect (at 2.45 -1.6 225) (size 1.5 1) (layers "F.Cu" "F.Paste" "F.Mask")
-      (net 11 "Net-(D1-Pad2)") (pinfunction "DIN") (pintype "input"))
+      (net 10 "Net-(D1-Pad2)") (pinfunction "DIN") (pintype "input"))
     (model "${KICAD6_3DMODEL_DIR}/LED_SMD.3dshapes/LED_WS2812B_PLCC4_5.0x5.0mm_P3.2mm.wrl"
       (offset (xyz 0 0 0))
@@
     )
     (pad "1" smd rect (at -7.08 0 180) (size 1.5 3.8) (layers "B.Cu" "B.Paste" "B.Mask")
-      (net 7 "unconnected-(CN3-Pad1)") (pinfunction "1") (pintype "bidirectional") (solder_mask_margin 0.1016))
+      (net 2 "Net-(CN1-Pad1)") (pinfunction "1") (pintype "bidirectional") (solder_mask_margin 0.1016))
     (pad "2" smd rect (at -4.08 0 180) (size 1.5 3.8) (layers "B.Cu" "B.Paste" "B.Mask")
-      (net 8 "unconnected-(CN3-Pad2)") (pinfunction "2") (pintype "bidirectional") (solder_mask_margin 0.1016))
+      (net 3 "Net-(CN1-Pad2)") (pinfunction "2") (pintype "bidirectional") (solder_mask_margin 0.1016))
     (pad "3" smd rect (at -0.92 0 180) (size 1.5 3.8) (layers "B.Cu" "B.Paste" "B.Mask")
-      (net 9 "Net-(CN3-Pad3)") (pinfunction "3") (pintype "bidirectional") (solder_mask_margin 0.1016))
+      (net 8 "Net-(CN3-Pad3)") (pinfunction "3") (pintype "bidirectional") (solder_mask_margin 0.1016))
     (pad "4" smd rect (at 2.08 0 180) (size 1.5 3.8) (layers "B.Cu" "B.Paste" "B.Mask")
-      (net 10 "Net-(CN3-Pad4)") (pinfunction "4") (pintype "bidirectional") (solder_mask_margin 0.1016))
+      (net 9 "Net-(CN3-Pad4)") (pinfunction "4") (pintype "bidirectional") (solder_mask_margin 0.1016))
     (pad "5" smd rect (at 5.08 0 180) (size 1.5 3.8) (layers "B.Cu" "B.Paste" "B.Mask")
       (net 5 "+5V") (pinfunction "5") (pintype "bidirectional") (solder_mask_margin 0.1016))
@@
   (segment (start 125.984 99.87) (end 155.686 99.87) (width 0.25) (layer "B.Cu") (net 2))
   (segment (start 155.686 99.87) (end 155.702 99.854) (width 0.25) (layer "B.Cu") (net 2))
+  (segment (start 155.194 99.854) (end 148.304 92.964) (width 0.25) (layer "B.Cu") (net 2))
+  (segment (start 155.702 99.854) (end 155.194 99.854) (width 0.25) (layer "B.Cu") (net 2))
   (segment (start 155.702 102.854) (end 126 102.854) (width 0.25) (layer "B.Cu") (net 3))
+  (segment (start 156.852 102.854) (end 157.9302 101.7758) (width 0.25) (layer "B.Cu") (net 3))
+  (segment (start 145.7382 90.7358) (end 145.304 91.17) (width 0.25) (layer "B.Cu") (net 3))
+  (segment (start 155.702 102.854) (end 156.852 102.854) (width 0.25) (layer "B.Cu") (net 3))
+  (segment (start 157.9302 98.7482) (end 149.9178 90.7358) (width 0.25) (layer "B.Cu") (net 3))
+  (segment (start 145.304 91.17) (end 145.304 92.964) (width 0.25) (layer "B.Cu") (net 3))
   (segment (start 126 102.854) (end 125.984 102.87) (width 0.25) (layer "B.Cu") (net 3))
+  (segment (start 157.9302 101.7758) (end 157.9302 98.7482) (width 0.25) (layer "B.Cu") (net 3))
+  (segment (start 149.9178 90.7358) (end 145.7382 90.7358) (width 0.25) (layer "B.Cu") (net 3))
   (segment (start 156.882 107.024) (end 154.686 109.22) (width 0.25) (layer "F.Cu") (net 4))
   (segment (start 156.882 105.842) (end 156.882 107.024) (width 0.25) (layer "F.Cu") (net 4))
@@
   (via (at 125.984 112.014) (size 0.8) (drill 0.4) (layers "F.Cu" "B.Cu") (net 5))
   (via (at 124.714 108.966) (size 0.8) (drill 0.4) (layers "F.Cu" "B.Cu") (net 6))
-  (segment (start 142.316 97.446) (end 142.316 94.31) (width 0.25) (layer "F.Cu") (net 9))
-  (segment (start 142.316 94.31) (end 142.24 94.234) (width 0.25) (layer "F.Cu") (net 9))
-  (via (at 142.24 94.234) (size 0.8) (drill 0.4) (layers "F.Cu" "B.Cu") (net 9))
-  (via (at 139.192 92.71) (size 0.8) (drill 0.4) (layers "F.Cu" "B.Cu") (net 10))
-  (segment (start 129.704 105.842) (end 134.164741 105.842) (width 0.25) (layer "F.Cu") (net 11))
-  (segment (start 141.431477 99.752218) (end 143.694218 102.014959) (width 0.25) (layer "F.Cu") (net 12))
-  (segment (start 135.729041 99.752218) (end 141.431477 99.752218) (width 0.25) (layer "F.Cu") (net 12))
-  (segment (start 149.421782 103.217041) (end 149.421782 106.481782) (width 0.25) (layer "F.Cu") (net 13))
-  (segment (start 149.421782 106.481782) (end 151.982 109.042) (width 0.25) (layer "F.Cu") (net 13))
+  (segment (start 149.421782 103.217041) (end 149.421782 106.481782) (width 0.25) (layer "F.Cu") (net 7))
+  (segment (start 149.421782 106.481782) (end 151.982 109.042) (width 0.25) (layer "F.Cu") (net 7))
+  (segment (start 142.316 97.446) (end 142.316 94.31) (width 0.25) (layer "F.Cu") (net 8))
+  (segment (start 142.316 94.31) (end 142.24 94.234) (width 0.25) (layer "F.Cu") (net 8))
+  (via (at 142.24 94.234) (size 0.8) (drill 0.4) (layers "F.Cu" "B.Cu") (net 8))
+  (via (at 139.192 92.71) (size 0.8) (drill 0.4) (layers "F.Cu" "B.Cu") (net 9))
+  (segment (start 129.704 105.842) (end 134.164741 105.842) (width 0.25) (layer "F.Cu") (net 10))
+  (segment (start 141.431477 99.752218) (end 143.694218 102.014959) (width 0.25) (layer "F.Cu") (net 11))
+  (segment (start 135.729041 99.752218) (end 141.431477 99.752218) (width 0.25) (layer "F.Cu") (net 11))
   (zone (net 1) (net_name "GND") (layers F&B.Cu) (hatch edge 0.508)
     (priority 6)
