File: PCB Design/T intersection straight/Adafruit NeoPixel 8 Stick.kicad_sch (KiCad schematic)
At the start: 8 parts, among them CN1 1X4SMT, CN2 1X4SMT, CN3 1X4SMT

Commit message: changes
Connections:
- net at CN3.1: now also CN1.1, CN2.6
- net at CN3.2: now also CN1.2, CN2.5
Changed lines of the file:
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@@
   (junction (at 107.95 129.54) (diameter 0) (color 0 0 0 0)
   )
+  (junction (at 182.88 82.55) (diameter 0) (color 0 0 0 0)
+  )
   (junction (at 148.59 129.54) (diameter 0) (color 0 0 0 0)
+  )
+  (junction (at 171.45 86.36) (diameter 0) (color 0 0 0 0)
   )
   (junction (at 132.08 106.68) (diameter 0) (color 0 0 0 0)
@@
   )
   (junction (at 107.95 106.68) (diameter 0) (color 0 0 0 0)
+  )
+  (wire (pts (xy 154.94 153.67) (xy 154.94 123.19))
+    (stroke (width 0) (type default) (color 0 0 0 0))
   )
   (wire (pts (xy 163.83 161.29) (xy 168.91 161.29))
@@
     (stroke (width 0) (type default) (color 0 0 0 0))
   )
+  (wire (pts (xy 161.29 151.13) (xy 161.29 130.81))
+    (stroke (width 0) (type default) (color 0 0 0 0))
+  )
   (wire (pts (xy 139.7 114.3) (xy 140.97 114.3))
     (stroke (width 0) (type default) (color 0 0 0 0))
@@
     (stroke (width 0) (type default) (color 0 0 0 0))
   )
+  (wire (pts (xy 161.29 130.81) (xy 182.88 130.81))
+    (stroke (width 0) (type default) (color 0 0 0 0))
+  )
   (wire (pts (xy 107.95 106.68) (xy 132.08 106.68))
     (stroke (width 0) (type default) (color 0 0 0 0))
@@
   )
   (wire (pts (xy 73.66 114.3) (xy 100.33 114.3))
+    (stroke (width 0) (type default) (color 0 0 0 0))
+  )
+  (wire (pts (xy 171.45 86.36) (xy 250.19 86.36))
+    (stroke (width 0) (type default) (color 0 0 0 0))
+  )
+  (wire (pts (xy 171.45 123.19) (xy 171.45 86.36))
     (stroke (width 0) (type default) (color 0 0 0 0))
   )
@@
     (stroke (width 0) (type default) (color 0 0 0 0))
   )
-  (wire (pts (xy 38.1 82.55) (xy 255.27 82.55))
+  (wire (pts (xy 38.1 82.55) (xy 182.88 82.55))
     (stroke (width 0) (type default) (color 0 0 0 0))
   )
@@
     (stroke (width 0) (type default) (color 0 0 0 0))
   )
-  (wire (pts (xy 39.37 86.36) (xy 250.19 86.36))
+  (wire (pts (xy 39.37 86.36) (xy 171.45 86.36))
     (stroke (width 0) (type default) (color 0 0 0 0))
   )
@@
     (stroke (width 0) (type default) (color 0 0 0 0))
   )
+  (wire (pts (xy 182.88 82.55) (xy 255.27 82.55))
+    (stroke (width 0) (type default) (color 0 0 0 0))
+  )
   (wire (pts (xy 156.21 114.3) (xy 251.46 114.3))
     (stroke (width 0) (type default) (color 0 0 0 0))
@@
     (stroke (width 0) (type default) (color 0 0 0 0))
   )
+  (wire (pts (xy 154.94 123.19) (xy 171.45 123.19))
+    (stroke (width 0) (type default) (color 0 0 0 0))
+  )
   (wire (pts (xy 259.08 124.46) (xy 254 124.46))
     (stroke (width 0) (type default) (color 0 0 0 0))
   )
+  (wire (pts (xy 182.88 130.81) (xy 182.88 82.55))
+    (stroke (width 0) (type default) (color 0 0 0 0))
+  )
+  (wire (pts (xy 161.29 153.67) (xy 154.94 153.67))
+    (stroke (width 0) (type default) (color 0 0 0 0))
+  )
