File: PCB Design/T intersection straight right/Adafruit NeoPixel 8 Stick.kicad_sch (KiCad schematic)
At the start: 8 parts, among them CN1 1X4SMT, CN2 1X4SMT, CN3 1X4SMT

Commit message: t straight fix
Connections:
- net GND: now also CN3.3
- net at D4.2 (DOUT): no longer CN3.3
Changed lines of the file:
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@@
 (kicad_sch (version 20211123) (generator eeschema)
   (paper "A4")
+  (junction (at 161.29 163.83) (diameter 0) (color 0 0 0 0)
+  )
   (junction (at 148.59 106.68) (diameter 0) (color 0 0 0 0)
   )
@@
   )
   (wire (pts (xy 259.08 132.08) (xy 259.08 134.62))
+    (stroke (width 0) (type default) (color 0 0 0 0))
+  )
+  (wire (pts (xy 161.29 156.21) (xy 160.02 156.21))
     (stroke (width 0) (type default) (color 0 0 0 0))
   )
@@
     (stroke (width 0) (type default) (color 0 0 0 0))
   )
-  (wire (pts (xy 99.06 154.94) (xy 99.06 142.24))
-    (stroke (width 0) (type default) (color 0 0 0 0))
-  )
-  (wire (pts (xy 160.02 156.21) (xy 161.29 156.21))
-    (stroke (width 0) (type default) (color 0 0 0 0))
-  )
   (wire (pts (xy 250.19 86.36) (xy 250.19 121.92))
     (stroke (width 0) (type default) (color 0 0 0 0))
@@
     (stroke (width 0) (type default) (color 0 0 0 0))
   )
-  (wire (pts (xy 160.02 142.24) (xy 160.02 156.21))
-    (stroke (width 0) (type default) (color 0 0 0 0))
-  )
-  (wire (pts (xy 99.06 154.94) (xy 120.65 154.94))
-    (stroke (width 0) (type default) (color 0 0 0 0))
-  )
   (wire (pts (xy 107.95 121.92) (xy 107.95 129.54))
     (stroke (width 0) (type default) (color 0 0 0 0))
@@
   )
   (wire (pts (xy 250.19 121.92) (xy 259.08 121.92))
+    (stroke (width 0) (type default) (color 0 0 0 0))
+  )
+  (wire (pts (xy 160.02 156.21) (xy 160.02 163.83))
     (stroke (width 0) (type default) (color 0 0 0 0))
   )
@@
     (stroke (width 0) (type default) (color 0 0 0 0))
   )
-  (wire (pts (xy 99.06 142.24) (xy 160.02 142.24))
+  (wire (pts (xy 160.02 163.83) (xy 161.29 163.83))
     (stroke (width 0) (type default) (color 0 0 0 0))
   )
