File: PCB Design/argon mount/Adafruit NeoPixel 8 Stick.kicad_sch (KiCad schematic)
At the start: 2 parts, among them CN2 1X4SMT

Commit message: argon mount
Parts:
- added R1: R, Resistor_THT:R_Axial_DIN0207_L6.3mm_D2.5mm_P7.62mm_Horizontal, symbol Device:R
- added U1: MIC5219-2.85YM5, Package_TO_SOT_SMD:SOT-23-5, symbol Regulator_Linear:MIC5219-2.85YM5
- added U2: VL6180, Adafruit VL6180:VL6180, symbol Adafruit VL6180:VL6180
Connections:
- net +5V: now also U1.1 (IN), U1.3 (EN)
- net GND: now also U1.2 (GND), U2.12 (AVSS), U2.9 (AVSS_VCS)
- net at CN2.5, MD1.0 (P0.26/SDA): now also U2.6 (SDA)
- net at CN2.6, MD1.1 (P0.27/SCL): now also U2.5 (SCL)
- new net: R1.1, U1.5 (OUT), U2.10 (AVDD), U2.8 (AVDD_VCS)
- new net: R1.2, U2.4 (GPIO0)

Commit message: edited boards
Connections:
- net +5V: now also MD1.VBUS; no longer MD1.3.3V
Changed lines of the file:
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@@
     (pin "1")
   )
-  (symbol (lib_id "Adafruit NeoPixel 8 Stick-eagle-import:+5V") (at 68.58 100.33 90) (unit 1)
+  (symbol (lib_id "Adafruit NeoPixel 8 Stick-eagle-import:+5V") (at 68.58 105.41 90) (unit 1)
     (in_bom yes) (on_board yes)
-    (property "Reference" "#P+0101" (id 0) (at 68.58 100.33 0)
+    (property "Reference" "#P+0101" (id 0) (at 68.58 105.41 0)
       (effects (font (size 1.27 1.27)) hide)
     )
-    (property "Value" "+5V" (id 1) (at 73.66 102.87 90)
+    (property "Value" "+5V" (id 1) (at 73.66 107.95 90)
       (effects (font (size 1.778 1.5113)) (justify left bottom))
     )
-    (property "Footprint" "Adafruit NeoPixel 8 Stick:" (id 2) (at 68.58 100.33 0)
+    (property "Footprint" "Adafruit NeoPixel 8 Stick:" (id 2) (at 68.58 105.41 0)
       (effects (font (size 1.27 1.27)) hide)
     )
-    (property "Datasheet" "" (id 3) (at 68.58 100.33 0)
+    (property "Datasheet" "" (id 3) (at 68.58 105.41 0)
       (effects (font (size 1.27 1.27)) hide)
     )

Commit message: clean up boards + generate some gerber files
Connections:
- net SCL: now reaches CN2.6, MD1.1 (P0.27/SCL), U2.5 (SCL)
- net SDA: now reaches CN2.5, MD1.0 (P0.26/SDA), U2.6 (SDA)
- no-connect marks 0 -> 27
