File: PCB Design/blocked_intersection/blocked_intersection.kicad_sch (KiCad schematic)
At the start: 9 parts, among them CN1 1X4SMT, CN2 1X4SMT, CN3 1X4SMT, CN4 1X4SMT

Commit message: blocked intersection
Connections:
- net +5V: no longer CN1.5
- net GND: no longer CN1.3, CN1.6
- net at D5.2 (DOUT): now also CN4.4
- net at CN4.1: now also CN2.6, CN3.6
- net at CN4.2: now also CN2.5, CN3.5
- net at D3.2 (DOUT): no longer CN1.4
- now unconnected: CN1.1, CN1.2
- no-connect marks 3 -> 0
