File: PCB Design/microcontroller_th/microcontroller_th.kicad_pcb (KiCad board)
At the start: 2 copper layers, 34.5 x 47.5 mm, 9 parts, among them CN2 1X4SMT, U1 ATmega328P-P, Y1 Crystal_Small

Commit message: atmega reset
Connections:
- R1 pad 2: Net-(R1-Pad2) -> Net-(U1-Pad12)
- U1 pad 1: Net-(R1-Pad2) -> Net-(U1-Pad12)
- U1 pad 12: unconnected-(U1-Pad12) -> Net-(U1-Pad12)
Routing:
- net Net-(U1-Pad12): track 0.00 -> 43.3 mm, vias 0 -> 1
- net Net-(R1-Pad2): track 14.4 -> 0.00 mm, vias 1 -> 0

Commit message: mount fix + offshoot flip
Routing:
- net /SDA: track 33.3 -> 32.4 mm
- net /SCL: track 24.9 -> 24.2 mm
Other:
- outline, holes or cut-outs redrawn
Changed lines of the file:
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@@
     (property "Sheetfile" "microcontroller_th.kicad_sch")
     (property "Sheetname" "")
-    (fp_text reference "CN2" (at 11.684 -0.508 180) (layer "B.SilkS")
+    (fp_text reference "CN2" (at 14.0716 -0.3556 180) (layer "B.SilkS")
       (effects (font (size 1.27 1.27) (thickness 0.15)) (justify mirror))
     )
@@
       (net 5 "/SCL") (pinfunction "6") (pintype "bidirectional") (solder_mask_margin 0.1016))
   )
+  (gr_line (start 150.2 97.536001) (end 156.972 97.536) (layer "Edge.Cuts") (width 0.05))
+  (gr_line (start 129.2 97.536) (end 122.428 97.536) (layer "Edge.Cuts") (width 0.05))
   (gr_line (start 129.2 89.916) (end 150.2 89.916001) (layer "Edge.Cuts") (width 0.05))
   (gr_line (start 122.428 97.536) (end 122.428 137.414) (layer "Edge.Cuts") (width 0.05))
-  (gr_line (start 150.2 89.916001) (end 156.972 97.45) (layer "Edge.Cuts") (width 0.05))
+  (gr_line (start 150.2 89.916001) (end 150.2 97.536001) (layer "Edge.Cuts") (width 0.05))
   (gr_line (start 122.428 137.414) (end 156.972 137.414) (layer "Edge.Cuts") (width 0.05))
-  (gr_line (start 156.972 97.45) (end 156.972 137.414) (layer "Edge.Cuts") (width 0.05))
-  (gr_line (start 122.428 97.536) (end 129.2 89.916) (layer "Edge.Cuts") (width 0.05))
+  (gr_line (start 156.972 97.536) (end 156.972 137.414) (layer "Edge.Cuts") (width 0.05))
+  (gr_line (start 129.2 97.536) (end 129.2 89.916) (layer "Edge.Cuts") (width 0.05))
   (segment (start 138.644 110.196) (end 144.79 116.342) (width 0.25) (layer "F.Cu") (net 1))
   (segment (start 134.366 110.196) (end 138.644 110.196) (width 0.25) (layer "F.Cu") (net 1))
@@
   (segment (start 140.874 104.806) (end 140.874 93.726) (width 0.25) (layer "B.Cu") (net 3))
   (segment (start 144.79 108.722) (end 140.874 104.806) (width 0.25) (layer "B.Cu") (net 3))
-  (segment (start 153.5382 96.9238) (end 153.5382 102.5138) (width 0.25) (layer "B.Cu") (net 4))
-  (segment (start 148.1122 91.4978) (end 153.5382 96.9238) (width 0.25) (layer "B.Cu") (net 4))
+  (segment (start 136.7958 95.9542) (end 139.7578 95.9542) (width 0.25) (layer "B.Cu") (net 4))
   (segment (start 139.7958 91.4978) (end 148.1122 91.4978) (width 0.25) (layer "B.Cu") (net 4))
+  (segment (start 134.874 94.0324) (end 136.7958 95.9542) (width 0.25) (layer "B.Cu") (net 4))
+  (segment (start 149.0472 100.2792) (end 152.41 103.642) (width 0.25) (layer "B.Cu") (net 4))
+  (segment (start 148.1122 91.4978) (end 149.0472 92.4328) (width 0.25) (layer "B.Cu") (net 4))
+  (segment (start 139.7578 91.5358) (end 139.7958 91.4978) (width 0.25) (layer "B.Cu") (net 4))
   (segment (start 139.7578 95.9542) (end 139.7578 91.5358) (width 0.25) (layer "B.Cu") (net 4))
-  (segment (start 153.5382 102.5138) (end 152.41 103.642) (width 0.25) (layer "B.Cu") (net 4))
-  (segment (start 139.7578 91.5358) (end 139.7958 91.4978) (width 0.25) (layer "B.Cu") (net 4))
-  (segment (start 136.7958 95.9542) (end 139.7578 95.9542) (width 0.25) (layer "B.Cu") (net 4))
-  (segment (start 134.874 94.0324) (end 136.7958 95.9542) (width 0.25) (layer "B.Cu") (net 4))
+  (segment (start 149.0472 92.4328) (end 149.0472 100.2792) (width 0.25) (layer "B.Cu") (net 4))
   (segment (start 134.0782 92.9978) (end 133.35 93.726) (width 0.25) (layer "F.Cu") (net 5))
-  (segment (start 152.41 99.97063) (end 145.43717 92.9978) (width 0.25) (layer "F.Cu") (net 5))
-  (segment (start 145.43717 92.9978) (end 134.0782 92.9978) (width 0.25) (layer "F.Cu") (net 5))
-  (segment (start 152.41 101.102) (end 152.41 99.97063) (width 0.25) (layer "F.Cu") (net 5))
+  (segment (start 152.41 101.102) (end 150.632 101.102) (width 0.25) (layer "F.Cu") (net 5))
+  (segment (start 150.632 101.102) (end 142.5278 92.9978) (width 0.25) (layer "F.Cu") (net 5))
+  (segment (start 142.5278 92.9978) (end 134.0782 92.9978) (width 0.25) (layer "F.Cu") (net 5))
   (via (at 133.35 93.726) (size 0.8) (drill 0.4) (layers "F.Cu" "B.Cu") (net 5))
   (segment (start 133.35 93.726) (end 131.874 93.726) (width 0.25) (layer "B.Cu") (net 5))
