File: PCB Design/power_mount/power_mount.kicad_pcb (KiCad board)
At the start: 2 copper layers, 34.6 x 37.8 mm, 3 parts, among them CN2 1X4SMT, J1 PJ-102AH

Commit message: power pcb fix
Parts:
- moved CN2 1.01 mm to (138.9, 93.7), turned to 0 degrees
Routing:
- net +5V: track 47.6 -> 51.4 mm
Changed lines of the file:
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@@
   )
   (footprint "Adafruit NeoPixel 8 Stick:1X4-SMT" (layer "B.Cu")
-    (at 139.954 93.726 180)
+    (at 138.946 93.726)
     (property "Sheetfile" "Adafruit NeoPixel 8 Stick.kicad_sch")
     (property "Sheetname" "")
@@
       (effects (font (size 1.27 1.27) (thickness 0.15)) (justify mirror))
     )
-    (pad "1" smd rect (at -7.08 0 180) (size 1.5 3.8) (layers "B.Cu" "B.Paste" "B.Mask")
+    (pad "1" smd rect (at -7.08 0) (size 1.5 3.8) (layers "B.Cu" "B.Paste" "B.Mask")
       (net 2 "GND") (pinfunction "1") (pintype "bidirectional") (solder_mask_margin 0.1016))
-    (pad "2" smd rect (at -4.08 0 180) (size 1.5 3.8) (layers "B.Cu" "B.Paste" "B.Mask")
+    (pad "2" smd rect (at -4.08 0) (size 1.5 3.8) (layers "B.Cu" "B.Paste" "B.Mask")
       (net 1 "+5V") (pinfunction "2") (pintype "bidirectional") (solder_mask_margin 0.1016))
-    (pad "3" smd rect (at -0.92 0 180) (size 1.5 3.8) (layers "B.Cu" "B.Paste" "B.Mask")
+    (pad "3" smd rect (at -0.92 0) (size 1.5 3.8) (layers "B.Cu" "B.Paste" "B.Mask")
       (net 3 "unconnected-(CN2-Pad3)") (pinfunction "3") (pintype "bidirectional") (solder_mask_margin 0.1016))
-    (pad "4" smd rect (at 2.08 0 180) (size 1.5 3.8) (layers "B.Cu" "B.Paste" "B.Mask")
+    (pad "4" smd rect (at 2.08 0) (size 1.5 3.8) (layers "B.Cu" "B.Paste" "B.Mask")
       (net 2 "GND") (pinfunction "4") (pintype "bidirectional") (solder_mask_margin 0.1016))
-    (pad "5" smd rect (at 5.08 0 180) (size 1.5 3.8) (layers "B.Cu" "B.Paste" "B.Mask")
+    (pad "5" smd rect (at 5.08 0) (size 1.5 3.8) (layers "B.Cu" "B.Paste" "B.Mask")
       (net 4 "unconnected-(CN2-Pad5)") (pinfunction "5") (pintype "bidirectional") (solder_mask_margin 0.1016))
-    (pad "6" smd rect (at 8.08 0 180) (size 1.5 3.8) (layers "B.Cu" "B.Paste" "B.Mask")
+    (pad "6" smd rect (at 8.08 0) (size 1.5 3.8) (layers "B.Cu" "B.Paste" "B.Mask")
       (net 5 "unconnected-(CN2-Pad6)") (pinfunction "6") (pintype "bidirectional") (solder_mask_margin 0.1016))
   )
@@
   (segment (start 130.914 117.856) (end 145.266041 117.856) (width 0.25) (layer "F.Cu") (net 1))
   (segment (start 124.818 111.76) (end 130.914 117.856) (width 0.25) (layer "F.Cu") (net 1))
-  (segment (start 144.034 116.623959) (end 145.266041 117.856) (width 0.25) (layer "B.Cu") (net 1))
-  (segment (start 144.034 93.726) (end 144.034 116.623959) (width 0.25) (layer "B.Cu") (net 1))
+  (segment (start 134.866 107.455959) (end 145.266041 117.856) (width 0.25) (layer "B.Cu") (net 1))
+  (segment (start 134.866 93.726) (end 134.866 107.455959) (width 0.25) (layer "B.Cu") (net 1))
   (zone (net 2) (net_name "GND") (layers F&B.Cu) (hatch edge 0.508)
     (connect_pads (clearance 0.000001))

Commit message: mount fix + offshoot flip
Parts:
- moved CN2 0.25 mm to (139.2, 93.7)
Other:
- outline, holes or cut-outs redrawn
Changed lines of the file:
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@@
   )
   (footprint "Adafruit NeoPixel 8 Stick:1X4-SMT" (layer "B.Cu")
-    (at 138.946 93.726)
+    (at 139.2 93.726)
     (property "Sheetfile" "Adafruit NeoPixel 8 Stick.kicad_sch")
     (property "Sheetname" "")
@@
   (gr_line (start 130.048 89.915998) (end 149.352 89.915999) (layer "Edge.Cuts") (width 0.05))
   (gr_line (start 122.428 97.536) (end 122.428 127.762) (layer "Edge.Cuts") (width 0.05))
-  (gr_line (start 149.352 89.915999) (end 156.972 97.45) (layer "Edge.Cuts") (width 0.05))
+  (gr_line (start 149.352 89.915999) (end 149.352 97.535999) (layer "Edge.Cuts") (width 0.05))
   (gr_line (start 122.428 127.762) (end 157.054 127.762) (layer "Edge.Cuts") (width 0.05))
-  (gr_line (start 156.972 97.45) (end 157.054 127.762) (layer "Edge.Cuts") (width 0.05))
-  (gr_line (start 122.428 97.536) (end 130.048 89.915998) (layer "Edge.Cuts") (width 0.05))
+  (gr_line (start 156.972 97.536) (end 157.054 127.762) (layer "Edge.Cuts") (width 0.05))
+  (gr_line (start 130.048 97.535998) (end 122.428 97.536) (layer "Edge.Cuts") (width 0.05))
+  (gr_line (start 130.048 97.535998) (end 130.048 89.915998) (layer "Edge.Cuts") (width 0.05))
+  (gr_line (start 149.352 97.535999) (end 156.972 97.536) (layer "Edge.Cuts") (width 0.05))
   (segment (start 130.914 117.856) (end 145.266041 117.856) (width 0.25) (layer "F.Cu") (net 1))
   (segment (start 124.818 111.76) (end 130.914 117.856) (width 0.25) (layer "F.Cu") (net 1))
