File: PCB Design/straight_stick_offshoot_flipped/straight_stick_offshoot_flipped.kicad_pcb (KiCad board)
At the start: 2 copper layers, 72.5 x 26.1 mm, 11 parts, among them CN1 1X4SMT, CN2 1X4SMT, CN3 1X4SMT

Commit message: mount fix + offshoot flip
Parts:
- moved CN3 23.6 mm to (158.8, 119.9), turned to 180 degrees
Routing:
- net Net-(CN1-Pad1): track 79.6 -> 86.1 mm, vias 0 -> 2
- net +5V: track 96.8 -> 91.4 mm
- net Net-(CN1-Pad2): track 76.0 -> 80.1 mm, vias 2 -> 0
Other:
- board size 72.5 x 26.1 mm -> 72.5 x 26.2 mm
